File: cluster_ubs_dispatch/cluster_ubs_dispatch.kicad_pcb (KiCad board)
At the start: 2 copper layers, 253 x 84.5 mm, 15 parts, among them J1 USB_A_external, J10 USB_A_jetson_NC, J11 Conn_01x08_Pin, J2 USB_A_ard_leo_pico, J3 USB_A_jetson_NC2, J4 USB_A_jetson0, J5 USB_A_jetson1, J6 USB_A_jetson2, J7 USB_A_jetson3, J8 USB_A_jetson4, J9 USB_A_jetson5, U1 74HC4051, U2 74HC4051, U3 74HC4051, U4 74HC4051

Commit message: missing additional S connection
Parts:
- moved J11 86.7 mm to (140.9, 20.8)
- moved J1 53.7 mm to (102.0, 47.0)
- moved J2 53.5 mm to (102.0, 29.0)
- moved U1 49.6 mm to (141.6, 46.5), turned to -90 degrees
- moved U3 48.3 mm to (123.6, 46.5), turned to 90 degrees
- moved U2 47.2 mm to (141.1, 29.5), turned to -90 degrees
- moved U4 45.8 mm to (123.6, 29.5), turned to 90 degrees
- moved J8 35.5 mm to (268.5, 54.5)
- moved J9 35.0 mm to (286.0, 54.5)
- moved J3 34.5 mm to (268.5, 22.5)
- moved J10 34.0 mm to (286.0, 22.5)
- moved J5 8.00 mm to (165.0, 54.0)
- moved J6 8.00 mm to (183.5, 54.0)
Connections:
- J1 pad 4: /SHIELD -> /GND
- J11 pad 4: Net-(J11-Pin_4) -> /ENABLE_BARRE
- J11 pad 7: /ENABLE_BARRE -> /VEE
- U1 pad 1: Net-(J8-D+) -> Net-(J6-D+)
- U1 pad 13: Net-(J4-D+) -> Net-(J10-D+)
- U1 pad 14: Net-(J5-D+) -> Net-(J8-D+)
- U1 pad 15: Net-(J6-D+) -> Net-(J5-D+)
- U1 pad 2: Net-(J10-D+) -> Net-(J9-D+)
- U1 pad 5: Net-(J9-D+) -> Net-(J4-D+)
- U1 pad 6: Net-(J11-Pin_4) -> /ENABLE_BARRE
- U1 pad 7: /ENABLE_BARRE -> /VEE
- U2 pad 1: Net-(J8-D-) -> Net-(J4-D-)
- U2 pad 12: Net-(J7-D-) -> Net-(J5-D-)
- U2 pad 13: Net-(J4-D-) -> Net-(J8-D-)
- U2 pad 14: Net-(J5-D-) -> Net-(J10-D-)
- U2 pad 15: Net-(J6-D-) -> Net-(J3-D-)
- U2 pad 2: Net-(J10-D-) -> Net-(J7-D-)
- U2 pad 4: Net-(J3-D-) -> Net-(J9-D-)
- U2 pad 5: Net-(J9-D-) -> Net-(J6-D-)
- U2 pad 6: Net-(J11-Pin_4) -> /ENABLE_BARRE
- U2 pad 7: /ENABLE_BARRE -> /VEE
- U3 pad 10: Net-(J11-Pin_4) -> /ENABLE_BARRE
- U3 pad 6: Net-(J11-Pin_4) -> /ENABLE_BARRE
- U3 pad 7: /ENABLE_BARRE -> /VEE
- U3 pad 9: Net-(J11-Pin_4) -> /ENABLE_BARRE
- U4 pad 10: Net-(J11-Pin_4) -> /ENABLE_BARRE
- U4 pad 6: Net-(J11-Pin_4) -> /ENABLE_BARRE
- U4 pad 7: /ENABLE_BARRE -> /VEE
- U4 pad 9: Net-(J11-Pin_4) -> /ENABLE_BARRE
Routing:
- net /GND: track 0.00 -> 467.6 mm, vias 0 -> 400
- net Net-(J10-D+): track 0.00 -> 161.5 mm, vias 0 -> 2
- net Net-(J9-D-): track 0.00 -> 160.8 mm, vias 0 -> 2
- net Net-(J9-D+): track 0.00 -> 154.7 mm, vias 0 -> 2
- net Net-(J10-D-): track 0.00 -> 154.4 mm, vias 0 -> 2
- net Net-(J8-D+): track 0.00 -> 141.0 mm, vias 0 -> 2
- net Net-(J3-D+): track 0.00 -> 140.9 mm, vias 0 -> 2
- net Net-(J8-D-): track 0.00 -> 138.5 mm, vias 0 -> 2
- net Net-(J3-D-): track 0.00 -> 135.2 mm, vias 0 -> 2
- net Net-(J7-D+): track 0.00 -> 62.2 mm, vias 0 -> 4
- net /ENABLE_BARRE: track 0.00 -> 60.3 mm, vias 0 -> 7
- net Net-(J6-D-): track 0.00 -> 59.2 mm, vias 0 -> 2
- net Net-(J7-D-): track 0.00 -> 54.0 mm, vias 0 -> 2
- net /VEE: track 0.00 -> 53.9 mm, vias 0 -> 11
- net Net-(J6-D+): track 0.00 -> 47.1 mm, vias 0 -> 2
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- added copper zone on F.Cu, net /GND
- added copper zone on B.Cu, net /SHIELD
- added copper zone on F.Cu, net /SHIELD
- added copper zone on B.Cu, net /VCC
Other:
- board size 253 x 84.5 mm -> 200 x 44.5 mm
